Commit message: Update velodyne.xacro
added gazebo tag for sdformat_urdf to parse and convert the sensor tag to sdf correctly.

File: simulation/models/vehicle/velodyne.xacro (robot description, xacro)
@@ -12,5 +12,7 @@
             <inertia ixx="0.001" ixy="0" ixz="0" iyy="0.001" iyz="0" izz="0.001"/>
         </inertial>
-        <sensor name='VLP-16' type='gpu_lidar'>"
+    </link>
+    <gazebo reference="velodyne">
+        <sensor name='VLP-16' type='gpu_lidar'>
             <topic>velodyne_points</topic>
             <update_rate>10</update_rate>
@@ -39,4 +41,4 @@
             <visualize>true</visualize>
         </sensor>
-    </link>
+    </gazebo>
 </robot>
