Commit message: Update depth_camera.xacro
updated values to match the current camera description in ads_dv.sdf

File: simulation/models/vehicle/depth_camera.xacro (robot description, xacro)
@@ -18,17 +18,18 @@
             <inertia ixx="0.001" ixy="0" ixz="0" iyy="0.001" iyz="0" izz="0.001"/>
         </inertial>
-        <sensor name="zed2i_depth_camera" type="depth_camera">
+        <sensor name="zed2i_depth_camera" type="rgbd_camera">
             <update_rate>30</update_rate>
-            <topic>/zed2i/depth_camera</topic>
+            <topic>zed2i/depth_camera</topic>
             <camera>
+                <camera_info_topic>camera_info</camera_info_topic>
                 <horizontal_fov>1.9198622</horizontal_fov> <!-- 110 degrees -->
                 <image>
-                    <width>1280</width>
-                    <height>720</height>
+                    <width>640</width>
+                    <height>480</height>
                     <format>R_FLOAT32</format>
                 </image>
                 <clip>
-                    <near>0.3</near>
-                    <far>20.0</far>
+                    <near>1.5</near>
+                    <far>35.0</far>
                 </clip>
                 <noise>
@@ -50,5 +51,5 @@
         <parent link="camera_link"/>
         <child link="camera_link_optical"/>
-        <origin xyz="0 0 0" rpy="-1.5707963267948966 0 -1.5707963267948966"/>
+        <origin xyz="0 0 0" rpy="0 0 0"/>
     </joint>
     <gazebo reference='camera_to_optical'>

Commit message: Update depth_camera.xacro
added logical camera

File: simulation/models/vehicle/depth_camera.xacro (robot description, xacro)
@@ -57,3 +57,50 @@
         <preserveFixedJoint>True</preserveFixedJoint>
     </gazebo>
+    <!-- Logical Camera -->
+    <link name='logical_camera_link'>
+        <inertial>
+            <mass value="0.001"/>
+            <inertia ixx="0.001" ixy="0" ixz="0" iyy="0.001" iyz="0" izz="0.001"/>
+        </inertial>
+        <sensor name='logical_camera' type='logical_camera'>
+            <update_rate>30</update_rate>
+            <topic>logical_camera</topic>
+            <always_on>true</always_on>
+            <visualize>true</visualize>
+            <enable_metrics>true</enable_metrics>
+            <logical_camera>
+            <near>1.5</near>
+            <far>35</far>
+            <aspect_ratio>1.333333333333333</aspect_ratio>
+            <horizontal_fov>1.9198622000000001</horizontal_fov>
+            </logical_camera>
+        </sensor>
+    </link>
+    <joint name='base_to_logical_camera' type='fixed'>
+        <parent link="base_link"/>
+        <child link="logical_camera_link"/>
+        <origin xyz="0.48649999999999999 0 0.67100000000000004" rpy="0 0 0"/>
+        <axis>
+            <dynamics>
+                <spring_reference>0</spring_reference>
+                <spring_stiffness>0</spring_stiffness>
+            </dynamics>
+            <xyz>0 0 1</xyz>
+            <limit>
+                <lower>-inf</lower>
+                <upper>inf</upper>
+            </limit>
+        </axis>
+        <physics>
+            <ode>
+                <limit>
+                <cfm>0</cfm>
+                <erp>0.20000000000000001</erp>
+                </limit>
+            </ode>
+        </physics>
+    </joint>
+    <gazebo reference='base_to_logical_camera'>
+        <preserveFixedJoint>True</preserveFixedJoint>
+    </gazebo>
 </robot>

Commit message: Update depth_camera.xacro
added gazebo tags for sdformat_urdf to parse the sensor tags.

File: simulation/models/vehicle/depth_camera.xacro (robot description, xacro)
@@ -18,4 +18,6 @@
             <inertia ixx="0.001" ixy="0" ixz="0" iyy="0.001" iyz="0" izz="0.001"/>
         </inertial>
+    </link>
+    <gazebo reference="camera_link_optical">
         <sensor name="zed2i_depth_camera" type="rgbd_camera">
             <gz_frame_id>camera_link_optical</gz_frame_id>
@@ -48,5 +50,5 @@
             </camera>
         </sensor>
-    </link>
+    </gazebo>
     <joint name="camera_to_optical" type="fixed">
         <parent link="camera_link"/>
@@ -63,4 +65,6 @@
             <inertia ixx="0.001" ixy="0" ixz="0" iyy="0.001" iyz="0" izz="0.001"/>
         </inertial>
+    </link>
+    <gazebo reference='logical_camera_link'>
         <sensor name='logical_camera' type='logical_camera'>
             <update_rate>30</update_rate>
@@ -76,5 +80,5 @@
             </logical_camera>
         </sensor>
-    </link>
+    </gazebo>
     <joint name='base_to_logical_camera' type='fixed'>
         <parent link="base_link"/>
