Commit message: Update cone.sdf.xacro

File: simulation/models/cones/cone.sdf.xacro (robot description, xacro)
@@ -14,7 +14,4 @@
             <collision name="collision">
                 <geometry>
-                    <!-- <mesh>
-                        <uri>model://simulation/models/cones/cone_${type}/mesh.dae</uri>
-                    </mesh> -->
                     <!-- Simpler collision model for performance boost -->
                     <box>

Commit message: Updated cone collision values

File: simulation/models/cones/cone.sdf.xacro (robot description, xacro)
@@ -13,10 +13,21 @@
             </visual>
             <collision name="collision">
-                <geometry>
-                    <!-- Simpler collision model for performance boost -->
-                    <box>
-                        <size>0.2 0.2 0.5</size>
-                    </box>
-                </geometry>
+                <xacro:if value="${type == 'orange_big'}">
+                    <pose>0 0 0.232 0 0 0</pose>
+                    <geometry>
+                        <!-- Simpler collision model for performance boost -->
+                        <box>
+                            <size>0.26 0.26 0.53</size>
+                        </box>
+                    </geometry>
+                </xacro:if>
+                <xacro:unless value="${type == 'orange_big'}">
+                    <geometry>
+                        <!-- Simpler collision model for performance boost -->
+                        <box>
+                            <size>0.22 0.23 0.3</size>
+                        </box>
+                    </geometry>
+                </xacro:unless>
                 <surface>
                     <!-- Big performance boost by ignoring the friction of the cones-->
