Commit message: Update xacros to make cones top level models

File: simulation/models/cones/cone.sdf.xacro (robot description, xacro)
@@ -3,6 +3,11 @@
     <!-- Macro to define a cone -->
     <xacro:macro name="cone" params="name type pose">
-        <link name="${name}">
-            <pose>${pose}</pose>
+    <model name="${name}">
+        <static>true</static>
+        <plugin name="gz::sim::systems::PosePublisher" filename="gz-sim-pose-publisher-system">
+            <publish_model_pose>true</publish_model_pose>
+        </plugin>
+        <pose>${pose}</pose>
+        <link name="${name}_link">
             <visual name="visual">
                 <geometry>
@@ -70,4 +75,5 @@
             </inertial>
         </link>
+    </model>
     </xacro:macro>
 </robot>

File: simulation/models/tracks/acceleration.xacro (robot description, xacro)
@@ -72,82 +72,50 @@
     </model>
     <xacro:include filename="$(find simulation)/models/cones/cone.sdf.xacro"/>
-    <model name='blue_cones'>
-      <static>true</static>
-      <plugin name="gz::sim::systems::PosePublisher" filename="gz-sim-pose-publisher-system">
-        <use_pose_vector_msg>true</use_pose_vector_msg>
-        <publish_model_pose>true</publish_model_pose>
-        <publish_nested_model_pose>true</publish_nested_model_pose>
-      </plugin>
-      <xacro:cone name="blue_1" type="blue" pose="-45 1.5 0.15 0 0 0"/>
-      <xacro:cone name="blue_2" type="blue" pose="-40 1.5 0.15 0 0 0"/>
-      <xacro:cone name="blue_3" type="blue" pose="-35 1.5 0.15 0 0 0"/>
-      <xacro:cone name="blue_4" type="blue" pose="-30 1.5 0.15 0 0 0"/>
-      <xacro:cone name="blue_5" type="blue" pose="-25 1.5 0.15 0 0 0"/>
-      <xacro:cone name="blue_6" type="blue" pose="-20 1.5 0.15 0 0 0"/>
-      <xacro:cone name="blue_7" type="blue" pose="-15 1.5 0.15 0 0 0"/>
-      <xacro:cone name="blue_8" type="blue" pose="-10 1.5 0.15 0 0 0"/>
-      <xacro:cone name="blue_9" type="blue" pose="-5 1.5 0.15 0 0 0"/>
-      <xacro:cone name="blue_10" type="blue" pose="0 1.5 0.15 0 0 0"/>
-      <xacro:cone name="blue_11" type="blue" pose="5 1.5 0.15 0 0 0"/>
-      <xacro:cone name="blue_12" type="blue" pose="10 1.5 0.15 0 0 0"/>
-      <xacro:cone name="blue_13" type="blue" pose="15 1.5 0.15 0 0 0"/>
-      <xacro:cone name="blue_14" type="blue" pose="20 1.5 0.15 0 0 0"/>
-    </model>
-    <model name='yellow_cones'>
-      <static>true</static>
-      <plugin name="gz::sim::systems::PosePublisher" filename="gz-sim-pose-publisher-system">
-        <use_pose_vector_msg>true</use_pose_vector_msg>
-        <publish_model_pose>true</publish_model_pose>
-        <publish_nested_model_pose>true</publish_nested_model_pose>
-      </plugin>
-      <xacro:cone name="yellow_1" type="yellow" pose="-45 -1.5 0.15 0 0 0"/>
-      <xacro:cone name="yellow_2" type="yellow" pose="-40 -1.5 0.15 0 0 0"/>
-      <xacro:cone name="yellow_3" type="yellow" pose="-35 -1.5 0.15 0 0 0"/>
-      <xacro:cone name="yellow_4" type="yellow" pose="-30 -1.5 0.15 0 0 0"/>
-      <xacro:cone name="yellow_5" type="yellow" pose="-25 -1.5 0.15 0 0 0"/>
-      <xacro:cone name="yellow_6" type="yellow" pose="-20 -1.5 0.15 0 0 0"/>
-      <xacro:cone name="yellow_7" type="yellow" pose="-15 -1.5 0.15 0 0 0"/>
-      <xacro:cone name="yellow_8" type="yellow" pose="-10 -1.5 0.15 0 0 0"/>
-      <xacro:cone name="yellow_9" type="yellow" pose="-5 -1.5 0.15 0 0 0"/>
-      <xacro:cone name="yellow_10" type="yellow" pose="0 -1.5 0.15 0 0 0"/>
-      <xacro:cone name="yellow_11" type="yellow" pose="5 -1.5 0.15 0 0 0"/>
-      <xacro:cone name="yellow_12" type="yellow" pose="10 -1.5 0.15 0 0 0"/>
-      <xacro:cone name="yellow_13" type="yellow" pose="15 -1.5 0.15 0 0 0"/>
-      <xacro:cone name="yellow_14" type="yellow" pose="20 -1.5 0.15 0 0 0"/>
-    </model>
-    <model name='orange_cones'>
-      <static>true</static>
-      <plugin name="gz::sim::systems::PosePublisher" filename="gz-sim-pose-publisher-system">
-        <use_pose_vector_msg>true</use_pose_vector_msg>
-        <publish_model_pose>true</publish_model_pose>
-        <publish_nested_model_pose>true</publish_nested_model_pose>
-      </plugin>
-      <xacro:cone name="orange_1" type="orange" pose="30 1.5 0.15 0 0 0"/>
-      <xacro:cone name="orange_2" type="orange" pose="30 -1.5 0.15 0 0 0"/>
-      <xacro:cone name="orange_3" type="orange" pose="35 1.5 0.15 0 0 0"/>
-      <xacro:cone name="orange_4" type="orange" pose="35 -1.5 0.15 0 0 0"/>
-      <xacro:cone name="orange_5" type="orange" pose="40 1.5 0.15 0 0 0"/>
-      <xacro:cone name="orange_6" type="orange" pose="40 -1.5 0.15 0 0 0"/>
-      <xacro:cone name="orange_7" type="orange" pose="45 1.5 0.15 0 0 0"/>
-      <xacro:cone name="orange_8" type="orange" pose="45 -1.5 0.15 0 0 0"/>
-      <xacro:cone name="orange_9" type="orange" pose="50 1.5 0.15 0 0 0"/>
-      <xacro:cone name="orange_10" type="orange" pose="50 -1.5 0.15 0 0 0"/>
-      <xacro:cone name="orange_11" type="orange" pose="50 0.75 0.15 0 0 0"/>
-      <xacro:cone name="orange_12" type="orange" pose="50 -0.75 0.15 0 0 0"/>
-    </model>
-    <model name='big_orange_cones'>
-      <static>true</static>
-      <plugin name="gz::sim::systems::PosePublisher" filename="gz-sim-pose-publisher-system">
-        <use_pose_vector_msg>true</use_pose_vector_msg>
-        <publish_model_pose>true</publish_model_pose>
-        <publish_nested_model_pose>true</publish_nested_model_pose>
-      </plugin>
-      <xacro:cone name="orange_big_1" type="orange_big" pose="-50 1.5 0.033 0 0 0"/>
-      <xacro:cone name="orange_big_2" type="orange_big" pose="-50 -1.5 0.033 0 0 0"/>
-      <xacro:cone name="orange_big_3" type="orange_big" pose="-50.5 1.5 0.033 0 0 0"/>
-      <xacro:cone name="orange_big_4" type="orange_big" pose="-50.5 -1.5 0.033 0 0 0"/>
-      <xacro:cone name="orange_big_5" type="orange_big" pose="25 1.5 0.033 0 0 0"/>
-      <xacro:cone name="orange_big_6" type="orange_big" pose="25 -1.5 0.033 0 0 0"/>
-    </model>
+    <xacro:cone name="blue_1" type="blue" pose="-45 1.5 0.15 0 0 0"/>
+    <xacro:cone name="blue_2" type="blue" pose="-40 1.5 0.15 0 0 0"/>
+    <xacro:cone name="blue_3" type="blue" pose="-35 1.5 0.15 0 0 0"/>
+    <xacro:cone name="blue_4" type="blue" pose="-30 1.5 0.15 0 0 0"/>
+    <xacro:cone name="blue_5" type="blue" pose="-25 1.5 0.15 0 0 0"/>
+    <xacro:cone name="blue_6" type="blue" pose="-20 1.5 0.15 0 0 0"/>
+    <xacro:cone name="blue_7" type="blue" pose="-15 1.5 0.15 0 0 0"/>
+    <xacro:cone name="blue_8" type="blue" pose="-10 1.5 0.15 0 0 0"/>
+    <xacro:cone name="blue_9" type="blue" pose="-5 1.5 0.15 0 0 0"/>
+    <xacro:cone name="blue_10" type="blue" pose="0 1.5 0.15 0 0 0"/>
+    <xacro:cone name="blue_11" type="blue" pose="5 1.5 0.15 0 0 0"/>
+    <xacro:cone name="blue_12" type="blue" pose="10 1.5 0.15 0 0 0"/>
+    <xacro:cone name="blue_13" type="blue" pose="15 1.5 0.15 0 0 0"/>
+    <xacro:cone name="blue_14" type="blue" pose="20 1.5 0.15 0 0 0"/>
+    <xacro:cone name="yellow_1" type="yellow" pose="-45 -1.5 0.15 0 0 0"/>
+    <xacro:cone name="yellow_2" type="yellow" pose="-40 -1.5 0.15 0 0 0"/>
+    <xacro:cone name="yellow_3" type="yellow" pose="-35 -1.5 0.15 0 0 0"/>
+    <xacro:cone name="yellow_4" type="yellow" pose="-30 -1.5 0.15 0 0 0"/>
+    <xacro:cone name="yellow_5" type="yellow" pose="-25 -1.5 0.15 0 0 0"/>
+    <xacro:cone name="yellow_6" type="yellow" pose="-20 -1.5 0.15 0 0 0"/>
+    <xacro:cone name="yellow_7" type="yellow" pose="-15 -1.5 0.15 0 0 0"/>
+    <xacro:cone name="yellow_8" type="yellow" pose="-10 -1.5 0.15 0 0 0"/>
+    <xacro:cone name="yellow_9" type="yellow" pose="-5 -1.5 0.15 0 0 0"/>
+    <xacro:cone name="yellow_10" type="yellow" pose="0 -1.5 0.15 0 0 0"/>
+    <xacro:cone name="yellow_11" type="yellow" pose="5 -1.5 0.15 0 0 0"/>
+    <xacro:cone name="yellow_12" type="yellow" pose="10 -1.5 0.15 0 0 0"/>
+    <xacro:cone name="yellow_13" type="yellow" pose="15 -1.5 0.15 0 0 0"/>
+    <xacro:cone name="yellow_14" type="yellow" pose="20 -1.5 0.15 0 0 0"/>
+    <xacro:cone name="orange_1" type="orange" pose="30 1.5 0.15 0 0 0"/>
+    <xacro:cone name="orange_2" type="orange" pose="30 -1.5 0.15 0 0 0"/>
+    <xacro:cone name="orange_3" type="orange" pose="35 1.5 0.15 0 0 0"/>
+    <xacro:cone name="orange_4" type="orange" pose="35 -1.5 0.15 0 0 0"/>
+    <xacro:cone name="orange_5" type="orange" pose="40 1.5 0.15 0 0 0"/>
+    <xacro:cone name="orange_6" type="orange" pose="40 -1.5 0.15 0 0 0"/>
+    <xacro:cone name="orange_7" type="orange" pose="45 1.5 0.15 0 0 0"/>
+    <xacro:cone name="orange_8" type="orange" pose="45 -1.5 0.15 0 0 0"/>
+    <xacro:cone name="orange_9" type="orange" pose="50 1.5 0.15 0 0 0"/>
+    <xacro:cone name="orange_10" type="orange" pose="50 -1.5 0.15 0 0 0"/>
+    <xacro:cone name="orange_11" type="orange" pose="50 0.75 0.15 0 0 0"/>
+    <xacro:cone name="orange_12" type="orange" pose="50 -0.75 0.15 0 0 0"/>
+    <xacro:cone name="large_orange_1" type="large_orange" pose="-50 1.5 0.033 0 0 0"/>
+    <xacro:cone name="large_orange_2" type="large_orange" pose="-50 -1.5 0.033 0 0 0"/>
+    <xacro:cone name="large_orange_3" type="large_orange" pose="-50.5 1.5 0.033 0 0 0"/>
+    <xacro:cone name="large_orange_4" type="large_orange" pose="-50.5 -1.5 0.033 0 0 0"/>
+    <xacro:cone name="large_orange_5" type="large_orange" pose="25 1.5 0.033 0 0 0"/>
+    <xacro:cone name="large_orange_6" type="large_orange" pose="25 -1.5 0.033 0 0 0"/>
   </world>
 </sdf>

File: simulation/models/tracks/skidpad.xacro (robot description, xacro)
@@ -161,8 +161,8 @@
     <model name='big_orange_cones'>
       <static>true</static>
-      <xacro:cone name="orange_big_1" type="orange_big" pose="-1.783 1.4851 0.033 0 0 0"/>
-      <xacro:cone name="orange_big_2" type="orange_big" pose="-1.783 -1.485 0.033 0 0 0"/>
-      <xacro:cone name="orange_big_3" type="orange_big" pose="1.7837 1.4851 0.033 0 0 0"/>
-      <xacro:cone name="orange_big_4" type="orange_big" pose="1.7837 -1.485 0.033 0 0 0"/>
+      <xacro:cone name="large_orange_1" type="large_orange" pose="-1.783 1.4851 0.033 0 0 0"/>
+      <xacro:cone name="large_orange_2" type="large_orange" pose="-1.783 -1.485 0.033 0 0 0"/>
+      <xacro:cone name="large_orange_3" type="large_orange" pose="1.7837 1.4851 0.033 0 0 0"/>
+      <xacro:cone name="large_orange_4" type="large_orange" pose="1.7837 -1.485 0.033 0 0 0"/>
     </model>
   </world>

File: simulation/models/tracks/track_small.xacro (robot description, xacro)
@@ -61,85 +61,76 @@
     </model>
     <xacro:include filename="$(find simulation)/models/cones/cone.sdf.xacro"/>
-    <model name='blue_cones'>
-      <static>true</static>
-      <xacro:cone name="blue_1" type="blue" pose="-17.0129 9.72719 0.15 0 0 0"/>
-      <xacro:cone name="blue_2" type="blue" pose="-12.7541 12.8712 0.15 0 0 0"/>
-      <xacro:cone name="blue_3" type="blue" pose="-8.31569 13.0924 0.15 0 0 0"/>
-      <xacro:cone name="blue_4" type="blue" pose="9.62956 15.8379 0.15 0 0 0"/>
-      <xacro:cone name="blue_5" type="blue" pose="12.492 17.0404 0.15 0 0 0"/>
-      <xacro:cone name="blue_6" type="blue" pose="15.1389 16.5025 0.15 0 0 0"/>
-      <xacro:cone name="blue_7" type="blue" pose="19.5034 13.6361 0.15 0 0 0"/>
-      <xacro:cone name="blue_8" type="blue" pose="20.8922 11.7012 0.15 0 0 0"/>
-      <xacro:cone name="blue_9" type="blue" pose="17.5221 15.3812 0.15 0 0 0"/>
-      <xacro:cone name="blue_10" type="blue" pose="21.4761 8.79574 0.15 0 0 0"/>
-      <xacro:cone name="blue_11" type="blue" pose="20.9992 5.27662 0.15 0 0 0"/>
-      <xacro:cone name="blue_12" type="blue" pose="19.9925 2.24053 0.15 0 0 0"/>
-      <xacro:cone name="blue_13" type="blue" pose="19.0983 -0.671871 0.15 0 0 0"/>
-      <xacro:cone name="blue_14" type="blue" pose="17.1824 -3.23994 0.15 0 0 0"/>
-      <xacro:cone name="blue_15" type="blue" pose="11.114 -6.74408 0.15 0 0 0"/>
-      <xacro:cone name="blue_16" type="blue" pose="-4.06552 13.3637 0.15 0 0 0"/>
-      <xacro:cone name="blue_17" type="blue" pose="14.2831 -5.26437 0.15 0 0 0"/>
-      <xacro:cone name="blue_18" type="blue" pose="8.25363 -8.53889 0.15 0 0 0"/>
-      <xacro:cone name="blue_19" type="blue" pose="5.06185 -10.1551 0.15 0 0 0"/>
-      <xacro:cone name="blue_20" type="blue" pose="1.42086 -11.9634 0.15 0 0 0"/>
-      <xacro:cone name="blue_21" type="blue" pose="-2.4975 -14.0305 0.15 0 0 0"/>
-      <xacro:cone name="blue_22" type="blue" pose="-5.74864 -16.1217 0.15 0 0 0"/>
-      <xacro:cone name="blue_23" type="blue" pose="-9.34841 -17.1551 0.15 0 0 0"/>
-      <xacro:cone name="blue_24" type="blue" pose="-12.2114 -16.6459 0.15 0 0 0"/>
-      <xacro:cone name="blue_25" type="blue" pose="-14.4625 -14.9249 0.15 0 0 0"/>
-      <xacro:cone name="blue_26" type="blue" pose="-16.2427 -13.276 0.15 0 0 0"/>
-      <xacro:cone name="blue_27" type="blue" pose="-0.131239 13.3125 0.15 0 0 0"/>
-      <xacro:cone name="blue_28" type="blue" pose="-17.8615 -11.5349 0.15 0 0 0"/>
-      <xacro:cone name="blue_29" type="blue" pose="-19.1945 -8.52656 0.15 0 0 0"/>
-      <xacro:cone name="blue_30" type="blue" pose="-18.9382 -5.15509 0.15 0 0 0"/>
-      <xacro:cone name="blue_31" type="blue" pose="-18.8625 -4.02997 0.15 0 0 0"/>
-      <xacro:cone name="blue_32" type="blue" pose="-18.6872 -0.45783 0.15 0 0 0"/>
-      <xacro:cone name="blue_33" type="blue" pose="-18.1384 2.83132 0.15 0 0 0"/>
-      <xacro:cone name="blue_34" type="blue" pose="-17.8432 6.27091 0.15 0 0 0"/>
-      <xacro:cone name="blue_35" type="blue" pose="-15.5443 12.0063 0.15 0 0 0"/>
-      <xacro:cone name="blue_36" type="blue" pose="3.50416 13.7245 0.15 0 0 0"/>
-      <xacro:cone name="blue_37" type="blue" pose="7.13676 14.727 0.15 0 0 0"/>
-    </model>
-    <model name='yellow_cones'>
-      <static>true</static>
-      <xacro:cone name="yellow_1" type="yellow" pose="-12.2686 6.61784 0.15 0 0 0"/>
-      <xacro:cone name="yellow_2" type="yellow" pose="-9.65737 7.2378 0.15 0 0 0"/>
-      <xacro:cone name="yellow_3" type="yellow" pose="7.33516 9.03961 0.15 0 0 0"/>
-      <xacro:cone name="yellow_4" type="yellow" pose="10.548 10.5892 0.15 0 0 0"/>
-      <xacro:cone name="yellow_5" type="yellow" pose="13.1479 11.1316 0.15 0 0 0"/>
-      <xacro:cone name="yellow_6" type="yellow" pose="15.2725 10.0791 0.15 0 0 0"/>
-      <xacro:cone name="yellow_7" type="yellow" pose="16.8037 8.23821 0.15 0 0 0"/>
-      <xacro:cone name="yellow_8" type="yellow" pose="-6.90273 7.20128 0.15 0 0 0"/>
-      <xacro:cone name="yellow_9" type="yellow" pose="16.7063 6.10772 0.15 0 0 0"/>
-      <xacro:cone name="yellow_10" type="yellow" pose="15.876 3.47906 0.15 0 0 0"/>
-      <xacro:cone name="yellow_11" type="yellow" pose="15.106 1.5027 0.15 0 0 0"/>
-      <xacro:cone name="yellow_12" type="yellow" pose="13.6765 -0.472612 0.15 0 0 0"/>
-      <xacro:cone name="yellow_13" type="yellow" pose="9.41953 -2.84739 0.15 0 0 0"/>
-      <xacro:cone name="yellow_14" type="yellow" pose="12.0732 -1.43122 0.15 0 0 0"/>
-      <xacro:cone name="yellow_15" type="yellow" pose="7.26282 -3.9408 0.15 0 0 0"/>
-      <xacro:cone name="yellow_16" type="yellow" pose="4.65159 -5.15509 0.15 0 0 0"/>
-      <xacro:cone name="yellow_17" type="yellow" pose="1.78774 -6.66723 0.15 0 0 0"/>
-      <xacro:cone name="yellow_18" type="yellow" pose="-1.97969 -8.56329 0.15 0 0 0"/>
-      <xacro:cone name="yellow_19" type="yellow" pose="-3.80615 7.33616 0.15 0 0 0"/>
-      <xacro:cone name="yellow_20" type="yellow" pose="-5.18123 -10.5555 0.15 0 0 0"/>
-      <xacro:cone name="yellow_21" type="yellow" pose="-8.34841 -12.1551 0.15 0 0 0"/>
-      <xacro:cone name="yellow_22" type="yellow" pose="-9.78487 -11.8592 0.15 0 0 0"/>
-      <xacro:cone name="yellow_23" type="yellow" pose="-11.3484 -11.1551 0.15 0 0 0"/>
-      <xacro:cone name="yellow_24" type="yellow" pose="-13.2946 -8.64709 0.15 0 0 0"/>
-      <xacro:cone name="yellow_25" type="yellow" pose="-14.2998 -6.05581 0.15 0 0 0"/>
-      <xacro:cone name="yellow_26" type="yellow" pose="-14.0528 -3.05427 0.15 0 0 0"/>
-      <xacro:cone name="yellow_27" type="yellow" pose="-13.6807 -0.101053 0.15 0 0 0"/>
-      <xacro:cone name="yellow_28" type="yellow" pose="-13.3484 2.84491 0.15 0 0 0"/>
-      <xacro:cone name="yellow_29" type="yellow" pose="-0.595997 7.27843 0.15 0 0 0"/>
-      <xacro:cone name="yellow_30" type="yellow" pose="-13.3484 4.84491 0.15 0 0 0"/>
-      <xacro:cone name="yellow_31" type="yellow" pose="2.90884 7.57594 0.15 0 0 0"/>
-    </model>
-    <model name='big_orange_cones'>
-      <static>true</static>
-      <xacro:cone name="orange_big_1" type="orange_big" pose="1.14507 3.03746 0.033 0 0 0"/>
-      <xacro:cone name="orange_big_2" type="orange_big" pose="-0.919189 2.98971 0.033 0 0 0"/>
-      <xacro:cone name="orange_big_3" type="orange_big" pose="1.04889 -3.01482 0.033 0 0 0"/>
-      <xacro:cone name="orange_big_4" type="orange_big" pose="-1.21717 -3.06412 0.033 0 0 0"/>
-    </model>
+    <xacro:cone name="blue_1" type="blue" pose="-17.0129 9.72719 0.15 0 0 0"/>
+    <xacro:cone name="blue_2" type="blue" pose="-12.7541 12.8712 0.15 0 0 0"/>
+    <xacro:cone name="blue_3" type="blue" pose="-8.31569 13.0924 0.15 0 0 0"/>
+    <xacro:cone name="blue_4" type="blue" pose="9.62956 15.8379 0.15 0 0 0"/>
+    <xacro:cone name="blue_5" type="blue" pose="12.492 17.0404 0.15 0 0 0"/>
+    <xacro:cone name="blue_6" type="blue" pose="15.1389 16.5025 0.15 0 0 0"/>
+    <xacro:cone name="blue_7" type="blue" pose="19.5034 13.6361 0.15 0 0 0"/>
+    <xacro:cone name="blue_8" type="blue" pose="20.8922 11.7012 0.15 0 0 0"/>
+    <xacro:cone name="blue_9" type="blue" pose="17.5221 15.3812 0.15 0 0 0"/>
+    <xacro:cone name="blue_10" type="blue" pose="21.4761 8.79574 0.15 0 0 0"/>
+    <xacro:cone name="blue_11" type="blue" pose="20.9992 5.27662 0.15 0 0 0"/>
+    <xacro:cone name="blue_12" type="blue" pose="19.9925 2.24053 0.15 0 0 0"/>
+    <xacro:cone name="blue_13" type="blue" pose="19.0983 -0.671871 0.15 0 0 0"/>
+    <xacro:cone name="blue_14" type="blue" pose="17.1824 -3.23994 0.15 0 0 0"/>
+    <xacro:cone name="blue_15" type="blue" pose="11.114 -6.74408 0.15 0 0 0"/>
+    <xacro:cone name="blue_16" type="blue" pose="-4.06552 13.3637 0.15 0 0 0"/>
+    <xacro:cone name="blue_17" type="blue" pose="14.2831 -5.26437 0.15 0 0 0"/>
+    <xacro:cone name="blue_18" type="blue" pose="8.25363 -8.53889 0.15 0 0 0"/>
+    <xacro:cone name="blue_19" type="blue" pose="5.06185 -10.1551 0.15 0 0 0"/>
+    <xacro:cone name="blue_20" type="blue" pose="1.42086 -11.9634 0.15 0 0 0"/>
+    <xacro:cone name="blue_21" type="blue" pose="-2.4975 -14.0305 0.15 0 0 0"/>
+    <xacro:cone name="blue_22" type="blue" pose="-5.74864 -16.1217 0.15 0 0 0"/>
+    <xacro:cone name="blue_23" type="blue" pose="-9.34841 -17.1551 0.15 0 0 0"/>
+    <xacro:cone name="blue_24" type="blue" pose="-12.2114 -16.6459 0.15 0 0 0"/>
+    <xacro:cone name="blue_25" type="blue" pose="-14.4625 -14.9249 0.15 0 0 0"/>
+    <xacro:cone name="blue_26" type="blue" pose="-16.2427 -13.276 0.15 0 0 0"/>
+    <xacro:cone name="blue_27" type="blue" pose="-0.131239 13.3125 0.15 0 0 0"/>
+    <xacro:cone name="blue_28" type="blue" pose="-17.8615 -11.5349 0.15 0 0 0"/>
+    <xacro:cone name="blue_29" type="blue" pose="-19.1945 -8.52656 0.15 0 0 0"/>
+    <xacro:cone name="blue_30" type="blue" pose="-18.9382 -5.15509 0.15 0 0 0"/>
+    <xacro:cone name="blue_31" type="blue" pose="-18.8625 -4.02997 0.15 0 0 0"/>
+    <xacro:cone name="blue_32" type="blue" pose="-18.6872 -0.45783 0.15 0 0 0"/>
+    <xacro:cone name="blue_33" type="blue" pose="-18.1384 2.83132 0.15 0 0 0"/>
+    <xacro:cone name="blue_34" type="blue" pose="-17.8432 6.27091 0.15 0 0 0"/>
+    <xacro:cone name="blue_35" type="blue" pose="-15.5443 12.0063 0.15 0 0 0"/>
+    <xacro:cone name="blue_36" type="blue" pose="3.50416 13.7245 0.15 0 0 0"/>
+    <xacro:cone name="blue_37" type="blue" pose="7.13676 14.727 0.15 0 0 0"/>
+    <xacro:cone name="yellow_1" type="yellow" pose="-12.2686 6.61784 0.15 0 0 0"/>
+    <xacro:cone name="yellow_2" type="yellow" pose="-9.65737 7.2378 0.15 0 0 0"/>
+    <xacro:cone name="yellow_3" type="yellow" pose="7.33516 9.03961 0.15 0 0 0"/>
+    <xacro:cone name="yellow_4" type="yellow" pose="10.548 10.5892 0.15 0 0 0"/>
+    <xacro:cone name="yellow_5" type="yellow" pose="13.1479 11.1316 0.15 0 0 0"/>
+    <xacro:cone name="yellow_6" type="yellow" pose="15.2725 10.0791 0.15 0 0 0"/>
+    <xacro:cone name="yellow_7" type="yellow" pose="16.8037 8.23821 0.15 0 0 0"/>
+    <xacro:cone name="yellow_8" type="yellow" pose="-6.90273 7.20128 0.15 0 0 0"/>
+    <xacro:cone name="yellow_9" type="yellow" pose="16.7063 6.10772 0.15 0 0 0"/>
+    <xacro:cone name="yellow_10" type="yellow" pose="15.876 3.47906 0.15 0 0 0"/>
+    <xacro:cone name="yellow_11" type="yellow" pose="15.106 1.5027 0.15 0 0 0"/>
+    <xacro:cone name="yellow_12" type="yellow" pose="13.6765 -0.472612 0.15 0 0 0"/>
+    <xacro:cone name="yellow_13" type="yellow" pose="9.41953 -2.84739 0.15 0 0 0"/>
+    <xacro:cone name="yellow_14" type="yellow" pose="12.0732 -1.43122 0.15 0 0 0"/>
+    <xacro:cone name="yellow_15" type="yellow" pose="7.26282 -3.9408 0.15 0 0 0"/>
+    <xacro:cone name="yellow_16" type="yellow" pose="4.65159 -5.15509 0.15 0 0 0"/>
+    <xacro:cone name="yellow_17" type="yellow" pose="1.78774 -6.66723 0.15 0 0 0"/>
+    <xacro:cone name="yellow_18" type="yellow" pose="-1.97969 -8.56329 0.15 0 0 0"/>
+    <xacro:cone name="yellow_19" type="yellow" pose="-3.80615 7.33616 0.15 0 0 0"/>
+    <xacro:cone name="yellow_20" type="yellow" pose="-5.18123 -10.5555 0.15 0 0 0"/>
+    <xacro:cone name="yellow_21" type="yellow" pose="-8.34841 -12.1551 0.15 0 0 0"/>
+    <xacro:cone name="yellow_22" type="yellow" pose="-9.78487 -11.8592 0.15 0 0 0"/>
+    <xacro:cone name="yellow_23" type="yellow" pose="-11.3484 -11.1551 0.15 0 0 0"/>
+    <xacro:cone name="yellow_24" type="yellow" pose="-13.2946 -8.64709 0.15 0 0 0"/>
+    <xacro:cone name="yellow_25" type="yellow" pose="-14.2998 -6.05581 0.15 0 0 0"/>
+    <xacro:cone name="yellow_26" type="yellow" pose="-14.0528 -3.05427 0.15 0 0 0"/>
+    <xacro:cone name="yellow_27" type="yellow" pose="-13.6807 -0.101053 0.15 0 0 0"/>
+    <xacro:cone name="yellow_28" type="yellow" pose="-13.3484 2.84491 0.15 0 0 0"/>
+    <xacro:cone name="yellow_29" type="yellow" pose="-0.595997 7.27843 0.15 0 0 0"/>
+    <xacro:cone name="yellow_30" type="yellow" pose="-13.3484 4.84491 0.15 0 0 0"/>
+    <xacro:cone name="yellow_31" type="yellow" pose="2.90884 7.57594 0.15 0 0 0"/>
+    <xacro:cone name="orange_big_1" type="orange_big" pose="1.14507 3.03746 0.033 0 0 0"/>
+    <xacro:cone name="orange_big_2" type="orange_big" pose="-0.919189 2.98971 0.033 0 0 0"/>
+    <xacro:cone name="orange_big_3" type="orange_big" pose="1.04889 -3.01482 0.033 0 0 0"/>
+    <xacro:cone name="orange_big_4" type="orange_big" pose="-1.21717 -3.06412 0.033 0 0 0"/>
   </world>
 </sdf>
